File: kicad/esphome-pelletkachel/esphome-pelletkachel.kicad_sch (KiCad schematic)
At the start: 4 parts, among them J1 Display-MCU-Connector, J3 MOSI-RSTSKIMIS, J5 Wireless-Headers, U1 ESP32-DEVKITC-32U

Commit message: changed drawing
Parts:
- added D1: LED, symbol Device:LED
- added R18, R19: ~, symbol Connector_Generic:Conn_02x01
- J5: value Wireless-Headers -> ~
Connections:
- net +5V: now reaches U1.19 (EXT_5V)
- net +5V: now also J5.2 (Pin_2)
- net at J1.R (Pin_2): now also R19.2 (Pin_2)
- net at J1.T (Pin_1): now also R18.2 (Pin_2)
Other:
- note added: "?"
- note added: "GPIO16 <- TX PIN ON DISPLAY BOARD GPIO21 -> RX PIN " " " GPIO27 <- MCU CONTROL BOARD SENSOR FROM MCU GPIO25 -> AUGER OUT TO OPTOISOLATOR GPIO19 -> LED ON DISPLAY FRO P5 GPIO26 -> THUMBS UP RESET GPIO5 <-> SDA GPIO33 <-> SCL"
- note added: "To what header pins lead the R19 and R18 pads?"
- note added: "Where is GND?"
- note added: "Where is TuyaMCU TX and RX?"
- moved on the sheet: J5

Commit message: changed drawing
Connections:
- net GND: now also J5.4 (Pin_4), U1.38 (GND3)
- net RX - TuyaMCU: now reaches J5.10 (Pin_10)
- net TX - TuyaMCU: now reaches J5.12 (Pin_12)
- net Reset: now reaches J5.15 (Pin_15)
- net RX - Display (MOD): now reaches J5.6 (Pin_6)
- net TX - Display (MOD): now reaches J5.8 (Pin_8)
- net Timer LED: now reaches J5.9 (Pin_9)
Other:
- note added: "How is reset wired?"
- note removed: "?"

Commit message: some edits
Parts:
- added J2: Display-MCU-Connector, symbol Connector_Generic:Conn_01x04
- added JB1: J5 Even, symbol Connector_Generic:Conn_01x08
- added JB2: J5 Odd, symbol Connector_Generic:Conn_01x08
- added JB3: Thumbs, symbol Connector:Screw_Terminal_01x02
- added JB4: Mainboard (DPC), symbol Connector_Generic:Conn_01x04
- added JB5: Display (J1), symbol Connector_Generic:Conn_01x04
- added U2: 757, 757:MODULE_757, symbol 4ch-LLC:757
- D1, J1, J3, J5, R18, R19: now left out of the parts list
Connections:
- net +5V: now also JB4.V (Pin_4), JB5.V (Pin_4), U2.HV; no longer J5.2 (Pin_2)
- net GND: now also JB4.G (Pin_3), JB5.G (Pin_3), U2.GND_1 (GND), U2.GND_2 (GND); no longer J5.4 (Pin_4)
- net +3.3V: now reaches U1.1 (3V3)
- net +3.3V: now also U2.LV
- net at R19.2 (Pin_2): no longer J1.R (Pin_2)
- net at R18.2 (Pin_2): no longer J1.T (Pin_1)
- net RX - Display (MOD): no longer names the net of J5.6 (Pin_6)
- net Reset: no longer names the net of J5.15 (Pin_15)
- net TX - Display (MOD): no longer names the net of J5.8 (Pin_8)
- net Timer LED: no longer names the net of J5.9 (Pin_9)
- new net: JB4.R (Pin_2), JB5.R (Pin_2)
- new net: JB4.T (Pin_1), JB5.T (Pin_1)
Other:
- note added: "Mainboard"
- note removed: "GPIO16 <- TX PIN ON DISPLAY BOARD GPIO21 -> RX PIN " " " GPIO27 <- MCU CONTROL BOARD SENSOR FROM MCU GPIO25 -> AUGER OUT TO OPTOISOLATOR GPIO19 -> LED ON DISPLAY FRO P5 GPIO26 -> THUMBS UP RESET GPIO5 <-> SDA GPIO33 <-> SCL"
- note removed: "How is reset wired?"
- note removed: "To what header pins lead the R19 and R18 pads?"
- note removed: "Where is GND?"
- note removed: "Where is TuyaMCU TX and RX?"
- moved on the sheet: D1, J1, J3, J5, R18, R19

Commit message: completed schematic so far
Parts:
- added J4: Thumbs, symbol Connector_Generic:Conn_02x02_Row_Letter_Last
- added U3: VL53L0CXV0DH1, Sensor_Distance:ST_VL53L1x, symbol Sensor_Distance:VL53L0CXV0DH1
Connections:
- net +3.3V: now also U3.11 (AVDD)
- net +5V: now also JB1.1 (Pin_1)
- net GND: now also JB1.2 (Pin_2), U3.12 (GND), U3.3 (GND), U3.4 (GND), U3.6 (GND)
- net Reset: now reaches U1.10 (IO26)
- net Reset: now also JB3.1 (Pin_1)
- net MCU UART TX Read: now reaches U1.27 (IO16)
- net MCU UART TX Read: now also U2.LV1
- net MCU UART RX Read: now reaches U1.31 (IO19)
- net MCU UART RX Read: now also U2.LV2
- net SDA: now reaches U1.33 (IO21)
- net SDA: now also U3.9 (SDA)
- net RX to Display: now reaches U1.34 (RXD0)
- net RX to Display: now also U2.LV3
- net TX to Display: now reaches U1.35 (TXD0)
- net TX to Display: now also U2.LV4
- net SCL: now reaches U1.36 (IO22)
- net SCL: now also U3.10 (SCL)
- net at JB4.R (Pin_2), JB5.R (Pin_2): now also U2.HV2
- net at JB4.T (Pin_1), JB5.T (Pin_1): now also U2.HV1
- net RX to Display (HV): now reaches JB1.5 (Pin_5)
- net RX to Display (HV): now also U2.HV3
- net TX to Display (HV): now reaches JB1.6 (Pin_6)
- net TX to Display (HV): now also U2.HV4
Other:
- note added: "Connects to soldered wires on thumbs button (the not grounded side)"
- note added: "Display board connectors (J5)"
- note added: "Functionality description"
- note added: "Interconnects Display and Mainboard - Facilitates reading TX and RX lines by the ESP32 - Prevents soldering - Requires extra cable"
- note added: "Level Sensor VL53L0X"
- note added: "TX and RX to Display facilitates Tuya UART comms with display. Reading TX and RX lines between display and Mainboard facilitates: - message reading sent by display and - temp readings sent by mainboard Time of Flight sensor facilitates pellet container level."
- moved on the sheet: JB1, JB2, JB3, JB4, JB5

Commit message: improvements
Other:
- note added: "Interconnects Display and Mainboard - Facilitates reading TX and RX lines by the ESP32 Why? - Prevents soldering the display board - Requires extra cable"
- note removed: "Interconnects Display and Mainboard - Facilitates reading TX and RX lines by the ESP32 - Prevents soldering - Requires extra cable"
- company: (none) -> PITCon.nl
- title: (none) -> ESP32 Pellet Stove board
Changed lines of the file:
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@@
 	(generator_version "8.0")
 	(paper "A4")
+	(title_block
+		(title "ESP32 Pellet Stove board")
+		(date "2024-09-27")
+		(rev "v0.9")
+		(company "PITCon.nl")
+		(comment 1 "ESP32 PCB for pellet stove communication")
+	)
 		(symbol "Connector_Generic:Conn_02x05_Odd_Even"
 			(pin_names
@@
 		)
 	)
-	(text "Interconnects Display and Mainboard\n- Facilitates reading TX \n  and RX lines by the ESP32\n- Prevents soldering\n- Requires extra cable"
+	(text "Interconnects Display and Mainboard\n- Facilitates reading TX \n   and RX lines by the ESP32\n\nWhy?\n- Prevents soldering the \n   display board\n- Requires extra cable"
 		(exclude_from_sim no)
-		(at 95.758 180.086 0)
+		(at 95.25 182.88 0)
 		(effects
 			(font
@@
 		(on_board yes)
 		(dnp no)
-		(fields_autoplaced yes)
 		(property "Reference" "#PWR07"
 			(at 148.59 189.23 0)
@@
 		)
 		(property "Value" "+5V"
-			(at 156.21 189.2299 90)
+			(at 155.194 189.23 90)
 			(effects
 				(font
@@
 		(dnp no)
 		(property "Reference" "JB4"
-			(at 132.08 185.166 0)
+			(at 136.144 183.896 90)
 			(effects
 				(font
@@
 		)
 		(property "Value" "Mainboard (DPC)"
-			(at 132.08 187.706 0)
+			(at 138.684 183.896 90)
 			(effects
 				(font
@@
 		(dnp no)
 		(property "Reference" "JB5"
-			(at 166.116 184.912 0)
+			(at 160.782 181.864 90)
 			(effects
 				(font
@@
 		)
 		(property "Value" "Display (J1)"
-			(at 166.116 187.452 0)
+			(at 163.322 181.864 90)
 			(effects
 				(font
