File: kicad/esphome-pelletkachel/esphome-pelletkachel.kicad_pcb (KiCad board)
At the start: 2 copper layers, 48.3 x 106.7 mm, 7 parts, among them U1 ESP32-DEVKITC-32U, U3 VL53L0CXV0DH1

Commit message: this is hard
Parts:
- removed JB1: J5 Even, Connector_PinHeader_2.54mm:PinHeader_1x08_P2.54mm_Vertical
- removed JB2: J5 Odd, Connector_PinHeader_2.54mm:PinHeader_1x08_P2.54mm_Vertical
- removed JB3: Thumbs, TerminalBlock:TerminalBlock_bornier-2_P5.08mm
- removed JB4: Mainboard (DPC), Connector_JST:JST_XH_S4B-XH-A_1x04_P2.50mm_Horizontal
- removed JB5: Display (J1), Connector_JST:JST_XH_S4B-XH-A_1x04_P2.50mm_Horizontal
- removed U1: ESP32-DEVKITC-32U, ESP32-DEVKITC-32U:MODULE_ESP32-DEVKITC-32U
- removed U3: VL53L0CXV0DH1, Sensor_Distance:ST_VL53L1x
Other:
- board outline removed

Commit message: yac
Parts:
- added JB1: J5 Even, Connector_PinHeader_2.54mm:PinHeader_1x08_P2.54mm_Vertical, B.Cu at (102.2, 56.5)
- added JB2: J5 Odd, Connector_PinHeader_2.54mm:PinHeader_1x08_P2.54mm_Vertical, B.Cu at (76.8, 56.5)
- added JB3: Thumbs, TerminalBlock:TerminalBlock_bornier-2_P5.08mm, F.Cu at (76.2, 119.4)
- added JB4: Mainboard (DPC), Connector_JST:JST_XH_S4B-XH-A_1x04_P2.50mm_Horizontal, F.Cu at (94.0, 109.2)
- added JB5: Display (J1), Connector_JST:JST_XH_S4B-XH-A_1x04_P2.50mm_Horizontal, F.Cu at (81.3, 101.6)
- added JB6: To TOF, Connector_JST:JST_XH_S4B-XH-A_1x04_P2.50mm_Horizontal, F.Cu at (94.0, 124.3)
- added U1: ESP32-DEVKITC-32U, ESP32-DEVKITC-32U:MODULE_ESP32-DEVKITC-32U, F.Cu at (86.4, 71.1)
- added U2: 757, Ron-Custom-Components:TT-4chLLC-SKU000275, B.Cu at (76.2, 87.6)
Routing:
- added copper zone on B.Cu, net GND
Other:
- board outline added: 38.1 x 86.4 mm

Commit message: gefreubel
Parts:
- moved U2 32.3 mm to (103.1, 69.8), turned to 90 degrees
- moved JB5 26.1 mm to (95.9, 123.2), turned to 90 degrees
- moved JB6 26.1 mm to (81.0, 101.8), turned to -90 degrees
- moved JB4 1.91 mm to (95.9, 109.2)
Routing:
- net +5V: track 0.00 -> 104.7 mm
- net Net-(JB4-T): track 0.00 -> 69.2 mm, vias 0 -> 1
- net /SDA: track 0.00 -> 68.9 mm
- net /SCL: track 0.00 -> 68.4 mm
- net +3.3V: track 0.00 -> 61.6 mm
- net Net-(JB4-R): track 0.00 -> 54.6 mm
- net /LED: track 0.00 -> 50.3 mm
- net /Reset: track 0.00 -> 49.3 mm
- net /MCU UART RX Read: track 0.00 -> 20.6 mm
- net /RX to Display: track 0.00 -> 17.4 mm
- net /TX to Display: track 0.00 -> 17.4 mm
- net /MCU UART TX Read: track 0.00 -> 16.3 mm
- net /TX to Display (HV): track 0.00 -> 12.5 mm
- net /RX to Display (HV): track 0.00 -> 6.99 mm
Other:
- board text added: "${REFERENCE}"

Commit message: added tx rx switching method
Parts:
- added JP2: RX switcher, Connector_PinHeader_2.54mm:PinHeader_1x03_P2.54mm_Vertical, F.Cu at (131.2, 52.1)
- added JP3: TX switcher, Connector_PinHeader_2.54mm:PinHeader_1x03_P2.54mm_Vertical, F.Cu at (135.9, 52.1)
- added JP4: TX switcher, Connector_PinHeader_2.54mm:PinHeader_1x03_P2.54mm_Vertical, F.Cu at (145.8, 65.4)
- added JP5: RX switcher, Connector_PinHeader_2.54mm:PinHeader_1x03_P2.54mm_Vertical, F.Cu at (150.5, 65.4)
Connections:
- U2 pad 1: Net-(JB4-T) -> Net-(JP4-A)
- U2 pad 2: Net-(JB4-R) -> Net-(JP4-B)
- U2 pad 5: /RX to Display (HV) -> Net-(JP2-A)
- U2 pad 6: /TX to Display (HV) -> Net-(JP2-B)

Commit message: weer even uitgespeeld
Parts:
- added J6: 1-wire, Connector_PinHeader_2.54mm:PinHeader_1x03_P2.54mm_Vertical, F.Cu at (83.2, 47.0)
- added R1: 1k, Resistor_THT:R_Axial_DIN0204_L3.6mm_D1.6mm_P5.08mm_Horizontal, F.Cu at (87.6, 52.7)
- moved JP5 83.1 mm to (81.9, 112.4), turned to 180 degrees
- moved JP4 81.3 mm to (76.2, 107.3)
- moved JP2 72.8 mm to (71.8, 94.0), turned to 180 degrees
- moved JP3 70.0 mm to (71.8, 80.0)
- moved JB3 69.3 mm to (72.4, 50.2), turned to 0 degrees
- moved JB6 52.7 mm to (100.3, 52.7), turned to 180 degrees
- moved JB1 30.5 mm to (71.8, 57.1)
- moved JB5 20.6 mm to (75.6, 119.7), turned to 0 degrees
- moved JB2 20.3 mm to (97.2, 57.1)
- moved U2 19.3 mm to (87.6, 81.3), turned to 0 degrees
- moved JB4 10.6 mm to (92.7, 119.4), turned to 0 degrees
- moved U1 9.09 mm to (88.3, 80.0)
Connections:
- U1 pad 37: unconnected-(U1-IO23-Pad37) -> Net-(U1-IO23)
Routing:
- net /SCL: track 68.4 -> 14.6 mm
- net +5V: track 104.7 -> 154.5 mm
- net /SDA: track 68.9 -> 20.9 mm
- net Net-(JP2-A): track 0.00 -> 47.0 mm
- net Net-(JP4-B): track 0.00 -> 45.3 mm
- net Net-(JP4-A): track 0.00 -> 40.2 mm
- net Net-(JP2-B): track 0.00 -> 38.1 mm
- net Net-(JB4-T): track 69.2 -> 35.0 mm, vias 1 -> 0
- net Net-(JB4-R): track 54.6 -> 34.4 mm
- net /MCU UART TX Read: track 16.3 -> 35.8 mm
- net /RX to Display (HV): track 6.99 -> 26.2 mm, vias 0 -> 2
- net Net-(U1-IO23): track 0.00 -> 16.2 mm
- net /Reset: track 49.3 -> 33.8 mm, vias 0 -> 4
- net +3.3V: track 61.6 -> 46.7 mm
- net /LED: track 50.3 -> 37.2 mm, vias 0 -> 6
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Other:
- board text added: "+"
- board text added: "D"
- board text added: "Dallas"
- board text added: "Display"
- board text added: "G"
- board text added: "LED"
- board text added: "Level Indicator"
- board text added: "Mainboard"
- board text added: "Reset"
- board text added: "TX/RX MCU"
- board text removed: "${REFERENCE}"

Commit message: zooo
Parts:
- removed JP4: TX switcher, Connector_PinHeader_2.54mm:PinHeader_1x03_P2.54mm_Vertical
- removed JP5: RX switcher, Connector_PinHeader_2.54mm:PinHeader_1x03_P2.54mm_Vertical
- added G***: LOGO, LOGO, B.Cu at (94.0, 92.1)
- moved JB5 10.5 mm to (78.2, 109.6)
- moved JB4 9.80 mm to (92.8, 109.6)
Connections:
- JB4 pad 1: Net-(JB4-T) -> /MCUTX
- JB4 pad 2: Net-(JB4-R) -> /MCURX
- JB5 pad 1: Net-(JB4-T) -> /MCUTX
- JB5 pad 2: Net-(JB4-R) -> /MCURX
- U2 pad 1: Net-(JP4-A) -> /MCUTX
- U2 pad 2: Net-(JP4-B) -> /MCURX
Routing:
- net /MCURX: track 0.00 -> 59.2 mm
- net /MCUTX: track 0.00 -> 55.6 mm
- net Net-(JP4-B): track 45.3 -> 0.00 mm
- net Net-(JP4-A): track 40.2 -> 0.00 mm
- net Net-(JB4-T): track 35.0 -> 0.00 mm
- net Net-(JB4-R): track 34.4 -> 0.00 mm
- net +5V: track 154.5 -> 125.3 mm
Other:
- board size 38.1 x 86.4 mm -> 38.1 x 76.2 mm
- board text added: "1 2 3"
- board text added: "3 2 1"
- board text added: "PelletKachel PCB v2024.09.1.0"
- board text added: "R"
- board text added: "T"
- board text added: "V"
- board text removed: "TX/RX MCU"
