File: kicad/esphome-pelletkachel/esphome-pelletkachel.kicad_pcb (KiCad board)
At the start: 2 copper layers, 38.1 x 76.2 mm, 13 parts, among them J6 1-wire, U1 ESP32-DEVKITC-32U, U2 757

Commit message: changes
Parts:
- JP2, JP3: footprint Connector_PinHeader_2.54mm:PinHeader_1x03_P2.54mm_Vertical -> Jumper:SolderJumper-3_P1.3mm_Bridged12_RoundedPad1.0x1.5mm; moved to B.Cu
- moved JP3 21.6 mm to (86.0, 96.2), turned to 90 degrees
- moved JP2 11.2 mm to (82.7, 96.2), turned to -90 degrees
Routing:
- net +5V: track 125.3 -> 46.0 mm
- net /MCURX: track 59.2 -> 19.2 mm
- net /LED: track 37.2 -> 0.00 mm, vias 6 -> 0
- net /MCUTX: track 55.6 -> 19.5 mm
- net /MCU UART TX Read: track 35.8 -> 0.00 mm
- net /Reset: track 33.8 -> 0.00 mm, vias 4 -> 0
- net /RX to Display (HV): track 26.2 -> 0.00 mm, vias 2 -> 0
- net /MCU UART RX Read: track 25.0 -> 0.00 mm
- net /SDA: track 20.9 -> 0.00 mm
- net Net-(JP2-A): track 47.0 -> 26.4 mm
- net Net-(U1-IO23): track 16.2 -> 0.00 mm
- net /SCL: track 14.6 -> 0.00 mm
- net /TX to Display (HV): track 13.8 -> 0.00 mm
- net /RX to Display: track 12.4 -> 0.00 mm
- net /TX to Display: track 8.78 -> 0.00 mm
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Other:
- board text removed: "1 2 3"
- board text removed: "3 2 1"

Commit message: gedoe
Parts:
- moved R1 142.3 mm to (228.6, 33.0)
- moved J6 136.6 mm to (218.4, 27.9), turned to 90 degrees
- moved JB1 128.2 mm to (198.1, 35.6)
- moved JB2 128.2 mm to (223.5, 35.6)
- moved U2 126.3 mm to (212.1, 59.9)
- moved JB4 125.3 mm to (215.9, 86.4)
- moved JB5 124.8 mm to (200.8, 86.4)
- moved U1 122.4 mm to (208.3, 55.9)
- moved G*** 122.2 mm to (213.4, 66.0)
- moved JP3 121.6 mm to (205.7, 75.0)
- moved JP2 121.6 mm to (202.4, 75.0)
- moved JB6 78.4 mm to (176.5, 33.9)
- moved JB3 0.88 mm to (73.0, 49.5)
Routing:
- net +3.3V: track 47.0 -> 0.00 mm
- net +5V: track 46.0 -> 0.00 mm
- net Net-(JP2-B): track 30.1 -> 0.00 mm
- net Net-(JP2-A): track 26.4 -> 0.00 mm
- net /MCUTX: track 19.5 -> 0.00 mm
- net /MCURX: track 19.2 -> 0.00 mm
- removed copper zone on B.Cu, net GND
Other:
- board size 38.1 x 76.2 mm -> 40 x 70.5 mm

Commit message: changes
Parts:
- JB3: footprint TerminalBlock:TerminalBlock_bornier-2_P5.08mm -> TerminalBlock:TerminalBlock_Xinya_XY308-2.54-2P_1x02_P2.54mm_Horizontal
- moved JB3 126.9 mm to (195.7, 81.5)
- moved JB6 68.8 mm to (221.0, 86.4), turned to 90 degrees
- moved JP2 15.2 mm to (202.4, 59.7)
- moved JP3 15.2 mm to (205.7, 59.7)
- moved J6 10.5 mm to (228.6, 30.5), turned to -90 degrees
- moved JB5 9.23 mm to (195.6, 94.0)
- moved JB4 9.18 mm to (210.8, 94.0)
- moved R1 7.62 mm to (228.6, 40.6)
- moved G*** 5.68 mm to (210.8, 71.1)
- moved U1 5.68 mm to (205.7, 50.8)
Other:
- board size 40 x 70.5 mm -> 40 x 79.9 mm
- board text added: "Level"
- board text removed: "Level Indicator"

Commit message: changes
Parts:
- removed G***: LOGO, LOGO
- moved JB3 59.7 mm to (226.0, 30.0), turned to 180 degrees
- moved J6 55.5 mm to (213.4, 83.8)
- moved R1 44.4 mm to (205.7, 78.7), turned to 0 degrees
- moved JP3 21.6 mm to (198.1, 80.0)
- moved JP2 20.3 mm to (202.4, 80.0)
- moved JB6 7.63 mm to (220.7, 78.7), turned to 0 degrees
- moved JB4 1.42 mm to (209.4, 94.0)
- moved U2 1.27 mm to (210.8, 59.9)
Routing:
- net GND: track 0.00 -> 141.0 mm, vias 0 -> 8
- net +5V: track 0.00 -> 103.9 mm
- net +3.3V: track 0.00 -> 90.5 mm
- net /MCURX: track 0.00 -> 69.1 mm, vias 0 -> 1
- net /MCUTX: track 0.00 -> 55.7 mm, vias 0 -> 1
- net /LED: track 0.00 -> 55.1 mm
- net Net-(U1-IO23): track 0.00 -> 54.9 mm
- net /Reset: track 0.00 -> 53.4 mm
- net /SCL: track 0.00 -> 48.7 mm
- net /SDA: track 0.00 -> 40.1 mm
- net Net-(JP2-B): track 0.00 -> 39.2 mm
- net /RX to Display (HV): track 0.00 -> 38.0 mm, vias 0 -> 1
- net Net-(JP2-A): track 0.00 -> 35.2 mm
- net /TX to Display (HV): track 0.00 -> 34.9 mm, vias 0 -> 2
- net /MCU UART TX Read: track 0.00 -> 22.5 mm
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- added copper zone on B.Cu, net GND
Other:
- board size 40 x 79.9 mm -> 40.3 x 79.8 mm

Commit message: wat gefreubelt
Parts:
- moved JB6 45.6 mm to (210.7, 34.3), turned to 180 degrees
- moved JB3 30.5 mm to (195.6, 27.9), turned to -90 degrees
- moved J6 22.7 mm to (223.5, 63.5), turned to 180 degrees
- moved R1 18.9 mm to (223.5, 72.4), turned to 90 degrees
- moved JP3 15.3 mm to (213.3, 78.7), turned to 180 degrees
- moved JP2 13.3 mm to (213.3, 72.4), turned to 0 degrees
- moved U1 11.5 mm to (207.0, 62.2)
- moved U2 3.55 mm to (210.8, 63.5)
Routing:
- net GND: track 141.0 -> 0.00 mm, vias 8 -> 0
- net +5V: track 103.9 -> 0.00 mm
- net +3.3V: track 90.5 -> 0.00 mm
- net /MCURX: track 69.1 -> 0.00 mm, vias 1 -> 0
- net /MCUTX: track 55.7 -> 0.00 mm, vias 1 -> 0
- net /LED: track 55.1 -> 0.00 mm
- net Net-(U1-IO23): track 54.9 -> 0.00 mm
- net /Reset: track 53.4 -> 0.00 mm
- net /SCL: track 48.7 -> 0.00 mm
- net /SDA: track 40.1 -> 0.00 mm
- net Net-(JP2-B): track 39.2 -> 0.00 mm
- net /RX to Display (HV): track 38.0 -> 0.00 mm, vias 1 -> 0
- net Net-(JP2-A): track 35.2 -> 0.00 mm
- net /TX to Display (HV): track 34.9 -> 0.00 mm, vias 2 -> 0
- net /MCU UART TX Read: track 22.5 -> 0.00 mm
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
Commit message: beetje geschoven
Parts:
- moved JB3 1.27 mm to (195.6, 29.2)
Changed lines of the file:
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@@
 		(tags "Resistor Axial_DIN0204 series Axial Horizontal pin pitch 5.08mm 0.167W length 3.6mm diameter 1.6mm")
 		(property "Reference" "R1"
-			(at 2.413 0 90)
+			(at 2.54 1.778 90)
 			(layer "F.SilkS")
 			(effects
@@
 		(tags "connector JST XH horizontal")
 		(property "Reference" "JB6"
-			(at -4.5212 3.6576 90)
+			(at -4.184 3.81 90)
 			(layer "F.SilkS")
 			(effects
@@
 	(footprint "TerminalBlock:TerminalBlock_Xinya_XY308-2.54-2P_1x02_P2.54mm_Horizontal"
 		(layer "F.Cu")
-		(at 195.58 27.94 -90)
+		(at 195.58 29.21 -90)
 		(descr "Terminal Block Xinya XY308-2.54-2P, 2 pins, pitch 2.54mm, size 5.58x6.5mm^2, drill diameter 1.2mm, pad diameter 2mm, see http://www.xinyaelectronic.com/product/xy308-254, script-generated using https://gitlab.com/kicad/libraries/kicad-footprint-generator/-/tree/master/scripts/TerminalBlock_Xinya")
 		(tags "THT Terminal Block Xinya XY308-2.54-2P pitch 2.54mm size 5.58x6.5mm^2 drill 1.2mm pad 2mm")
 		(property "Reference" "JB3"
-			(at -3.0226 -3.5306 90)
+			(at -2.54 -3.048 180)
 			(layer "F.SilkS")
 			(effects
@@
 		(tags "connector JST XH horizontal")
 		(property "Reference" "JB4"
-			(at -1.524 -5.6388 0)
+			(at 0.9144 -4.826 0)
 			(layer "F.SilkS")
 			(effects
@@
 		(tags "connector JST XH horizontal")
 		(property "Reference" "JB5"
-			(at 0.9652 -5.588 180)
+			(at 1.524 -5.08 180)
 			(layer "F.SilkS")
 			(effects
@@
 		)
 		(fp_text user "${REFERENCE}"
-			(at 2.54 2.54 90)
+			(at -4.064 -0.508 90)
 			(layer "F.Fab")
 			(effects
@@
 	)
 	(gr_text "Reset"
-		(at 228.219 28.3972 -90)
+		(at 192.786 27.178 0)
 		(layer "F.SilkS")
 		(effects
@@
 	)
 	(gr_text "Mainboard"
-		(at 209.296 88.9508 0)
+		(at 212.09 89.662 0)
 		(layer "F.SilkS")
 		(effects
@@
 	)
 	(gr_text "PelletKachel PCB\nv2024.09.1.0"
-		(at 229.6668 54.7116 90)
+		(at 225.552 87.63 90)
 		(layer "F.SilkS")
 		(effects
@@
 	)
 	(gr_text "D"
-		(at 226.06 60.96 0)
+		(at 225.552 61.722 0)
 		(layer "F.SilkS")
 		(effects
@@
 	)
 	(gr_text "G"
-		(at 226.06 58.42 0)
+		(at 225.552 58.928 0)
 		(layer "F.SilkS")
 		(effects
@@
 	)
 	(gr_text "Display"
-		(at 198.12 88.9 0)
+		(at 198.628 89.408 0)
 		(layer "F.SilkS")
 		(effects
@@
 	)
 	(gr_text "Level"
-		(at 265.43 78.74 90)
+		(at 215.392 36.068 90)
 		(layer "F.SilkS")
 		(effects
@@
 	)
 	(gr_text "+"
-		(at 226.06 63.5 0)
+		(at 225.298 64.008 0)
 		(layer "F.SilkS")
 		(effects
@@
 	)
 	(gr_text "T"
-		(at 208.8896 91.2114 0)
+		(at 209.042 91.2114 0)
 		(layer "F.SilkS")
 		(effects
@@
 	)
 	(gr_text "G"
-		(at 200.54 91.08 0)
+		(at 199.898 91.08 0)
 		(layer "F.SilkS")
 		(effects
@@
 	)
 	(gr_text "V"
-		(at 203.08 91.08 0)
+		(at 202.692 91.08 0)
 		(layer "F.SilkS")
 		(effects
@@
 	)
 	(gr_text "Dallas"
-		(at 228.6 63.5 90)
+		(at 228.092 62.992 90)
 		(layer "F.SilkS")
 		(effects
@@
 	)
 	(gr_text "T"
-		(at 195.46 91.08 0)
+		(at 195.326 91.08 0)
 		(layer "F.SilkS")
 		(effects
@@
 	)
 	(gr_text "R"
-		(at 198 91.08 0)
+		(at 197.358 91.08 0)
 		(layer "F.SilkS")
 		(effects
@@
 	)
 	(gr_text "LED"
-		(at 221.3864 31.4198 90)
+		(at 195.58 34.29 180)
 		(layer "F.SilkS")
 		(effects
@@
 		(layer "F.Fab")
 		(pts
-			(xy 219.1324 105.2068) (xy 219.15 25.4)
+			(xy 217.753624 105.201107) (xy 217.771224 25.394307)
 		)
 		(height 25.814777)
 		(gr_text "79,8068 mm"
-			(at 243.805976 65.308839 89.98736441)
+			(at 242.4272 65.303146 89.98736441)
 			(layer "F.Fab")
 			(effects
